File: pitot/pitot.kicad_pcb (KiCad board)
At the start: 2 copper layers, 127 x 101.6 mm, 33 parts, among them IC1 LT1167CN8PBF, IC2 LT1167CN8PBF, IC3 LT1167CN8PBF, IC4 LTC1144CN8#PBF, IC5 DEV-11114, P1 DIL8, P2 DIL8, P3 DIL8, P4 CONN_01X04, U1 LM7809CT

Commit message: mkdir led AND pitot
Parts:
- moved C4 91.5 mm to (215.9, 83.8)
- moved C6 91.5 mm to (205.7, 83.8)
- moved D1 91.5 mm to (191.8, 86.4)
- moved P4 91.5 mm to (188.0, 99.1)
- moved R8 91.5 mm to (213.4, 86.4)
- moved C3 91.5 mm to (200.7, 83.8)
- moved C5 91.5 mm to (233.7, 83.8)
- moved C7 91.5 mm to (212.1, 83.8)
- moved C8 91.5 mm to (228.6, 83.8)
- moved D2 91.5 mm to (241.3, 91.4)
- moved D3 91.5 mm to (242.6, 86.4)
- moved IC2 91.5 mm to (223.5, 71.1)
- moved IC3 91.5 mm to (243.8, 71.1)
- moved IC5 91.5 mm to (198.1, 104.1)
- moved P1 91.5 mm to (200.7, 55.9)
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Routing:
- net Net-(C2-Pad2): track 76.5 -> 89.2 mm
- net Net-(IC1-Pad7): track 136.4 -> 135.1 mm
- net GND: track 398.4 -> 399.7 mm
- net +BATT: track 111.0 -> 109.7 mm
Other:
- board size 127 x 101.6 mm -> 162.6 x 63.5 mm
